Commit message: Update xacro macro use to follow conventions

File: urdf/heatsource_dynamic.urdf.xacro (robot description, xacro)
@@ -5,7 +5,7 @@
   xmlns:interface="http://www.ros.org/wiki/xacro"
   xmlns:xacro="http://www.ros.org/wiki/xacro">
-  <property name="M_PI" value="3.14159265359" />
-  <property name="offset_x" value="0" />
-  <property name="offset_y" value="0" />
+  <xacro:property name="M_PI" value="3.14159265359" />
+  <xacro:property name="offset_x" value="0" />
+  <xacro:property name="offset_y" value="0" />
   <xacro:include filename="$(find argo_objects_gazebo)/urdf/hotspot.urdf.xacro.xml" />
   <link name="world"/>

File: urdf/truss.urdf.xacro (robot description, xacro)
@@ -6,8 +6,8 @@
   xmlns:xacro="http://www.ros.org/wiki/xacro">
   <xacro:include filename="$(find hector_xacro_tools)/urdf/inertia_tensors.urdf.xacro" />
-  <macro name="truss_macro" params="name scale">
+  <xacro:macro name="truss_macro" params="name scale">
     <!--
     <joint name="${name}_joint" type="fixed">
-    <insert_block name="origin"/>
+    <xacro:insert_block name="origin"/>
     <parent link="${parent}" />
     <child link="${name}_link"/>
@@ -34,4 +34,4 @@
       <laserRetro>5003.0</laserRetro>
     </gazebo>
-  </macro>
+  </xacro:macro>
 </robot>
